File: pcb/bakeneko65ortho.kicad_pcb (KiCad board)
At the start: 2 copper layers, 303.8 x 94.2 mm, 165 parts, among them J1 1x4P 1mm, J2 AVR-ISP-6, SW1 SW_Push, U1 ATmega32U4-AU, U2 SRV05-4, Y1 16MHz

Commit message: add graphics
Parts:
- removed the G*** at (72.2, 50.0)
- removed J2: AVR-ISP-6, bakeneko:ISP
- added G***: LOGO, bakeneko65ortho:logo_4000_text, B.Cu at (32.6, 31.0)
- added G***: LOGO, bakeneko65ortho:drg_600_text_v2, F.Cu at (53.2, 54.2)
- moved F1 143.7 mm to (100.0, 30.4)
- moved U2 5.50 mm to (94.3, 28.2)
- moved R1 5.17 mm to (107.2, 29.2)
- moved R2 4.10 mm to (107.2, 27.2)
- moved C5 0.94 mm to (268.4, 40.4), turned to 90 degrees
- turned R4 to 180 degrees
Connections:
- R4 pad 1: GND -> Net-(R4-Pad1)
- R4 pad 2: Net-(R4-Pad2) -> GND
- U1 pad 10: MOSI -> Net-(U1-Pad10)
- U1 pad 11: MISO -> Net-(U1-Pad11)
- U1 pad 12: ROW1 -> Net-(U1-Pad12)
- U1 pad 33: Net-(R4-Pad2) -> Net-(R4-Pad1)
- U1 pad 9: SCK -> ROW1
Routing:
- net VBUS: track 178.6 -> 32.7 mm
- net +5V: track 125.4 -> 261.3 mm, vias 7 -> 6
- net MOSI: track 9.45 -> 0.00 mm
- net GND: track 377.9 -> 369.1 mm
- net SCK: track 7.42 -> 0.00 mm
- net RESET: track 32.4 -> 25.8 mm
- net /MCU_D-: track 165.3 -> 169.5 mm
- net /MCU_D+: track 166.0 -> 170.2 mm
- net MISO: track 4.20 -> 0.00 mm
- net Net-(R4-Pad2): track 3.90 -> 0.00 mm
- net Net-(R4-Pad1): track 0.00 -> 3.90 mm
- net D+: track 48.7 -> 45.8 mm
- net ROW1: track 294.8 -> 292.1 mm
- net D-: track 46.6 -> 44.0 mm
- net Net-(C5-Pad1): track 5.74 -> 3.80 mm
Other:
- net class USB: trace_width 0.2 -> 0.25
- board text removed: "Bakeneko65 Ortho"
